File: ai03-guide.sch (KiCad schematic (older format))
At the start: 24 parts, among them SW1 SW_Push, U1 ATmega32U4-AU, Y1 16MHz

Commit message: Routing
Connections:
- net COL0: now also U1.29 (PB5)
- net COL1: now also U1.28 (PB4)
- net ROW0: now also U1.30 (PB6)
- net ROW1: now also U1.27 (PD7)
Changed lines of the file:
@@
 EESchema Schematic File Version 4
+LIBS:ai03-guide-cache
 EELAYER 30 0
 EELAYER END
@@
 Text HLabel 8900 4350 0    50   Output ~ 0
 ROW1
+Text HLabel 6200 2350 2    50   Output ~ 0
+COL1
+Text HLabel 6200 2450 2    50   Output ~ 0
+COL0
+Text HLabel 6200 3850 2    50   Output ~ 0
+ROW1
+Text HLabel 6200 2550 2    50   Output ~ 0
+ROW0
 $EndSCHEMATC
