File: _autosave-ai03-guide.kicad_pcb (KiCad board)
At the start: 2 copper layers, 82 x 38.1 mm, 24 parts, among them SW1 SW_Push, U1 ATmega32U4-AU, Y1 16MHz

Commit message: Routing
Parts:
- C7: value 0.1uF -> 10uF
- moved C4 16.1 mm to (97.5, 107.0), turned to 180 degrees
- moved C3 14.2 mm to (112.1, 103.6)
- moved C2 13.2 mm to (95.0, 119.0), turned to 90 degrees
- moved C1 11.7 mm to (83.6, 119.0), turned to 270 degrees
- moved C7 1.35 mm to (91.9, 97.0)
- moved C5 1.10 mm to (78.7, 110.2)
- moved C6 0.84 mm to (84.0, 97.0)
- turned Y1 to 0 degrees
Routing:
- net GND: track 7.35 -> 46.8 mm
- net +5V: track 0.00 -> 23.9 mm
- net /COL0: track 0.00 -> 19.1 mm
- net /COL1: track 0.00 -> 19.0 mm
- net Net-(R2-Pad1): track 0.00 -> 17.1 mm
- net Net-(R3-Pad1): track 0.00 -> 15.3 mm
- net Net-(C2-Pad1): track 0.00 -> 13.9 mm
- net /ROW0: track 0.00 -> 13.1 mm
- net Net-(D3-Pad2): track 0.00 -> 13.1 mm
- net Net-(D4-Pad2): track 0.00 -> 12.9 mm
- net Net-(D1-Pad2): track 0.00 -> 12.7 mm
- net /ROW1: track 0.00 -> 12.2 mm
- net Net-(C1-Pad1): track 0.00 -> 10.3 mm
- net VCC: track 0.00 -> 7.47 mm
- net /D+: track 6.24 -> 7.19 mm

Commit message: Added Output
Parts:
- C7: value 10uF -> 0.1uF
Connections:
- U1 pad 27: Net-(U1-Pad27) -> /ROW1
- U1 pad 28: Net-(U1-Pad28) -> /COL1
- U1 pad 29: Net-(U1-Pad29) -> /COL0
- U1 pad 30: Net-(U1-Pad30) -> /ROW0
Routing:
- net +5V: track 23.9 -> 108.1 mm, vias 0 -> 8
- net GND: track 46.8 -> 115.8 mm
- net /COL0: track 19.1 -> 61.3 mm
- net Net-(R1-Pad2): track 0.00 -> 36.3 mm
- net Net-(R4-Pad2): track 0.00 -> 35.0 mm, vias 0 -> 2
- net /ROW1: track 12.2 -> 46.6 mm
- net /COL1: track 19.0 -> 41.9 mm
- net /ROW0: track 13.1 -> 33.1 mm
- net Net-(C3-Pad1): track 0.00 -> 19.8 mm
- added copper zone on B.Cu, net GND
Other:
- outline, holes or cut-outs redrawn
